File: UccMicroDuino/UccMicroDuino.kicad_pcb (KiCad board)
At the start: 2 copper layers, 8 parts, among them J1 Conn_01x10_Socket, J2 USB_A, U1 ATtiny85-20S

Commit message: Trabajo final
Parts:
- added D3: 3.6V 1/2 mW, Diode_SMD:D_SOD-123, F.Cu at (188.5, 85.5)
- added D4: Led Green, ledSmd:ledSMD, F.Cu at (197.0, 72.5)
- added R2: 68Ω 5% 1/8W, Resistor_SMD:R_0805_2012Metric_Pad1.20x1.40mm_HandSolder, F.Cu at (199.3, 84.0)
- added R3: 68Ω 5% 1/8W, Resistor_SMD:R_0805_2012Metric_Pad1.20x1.40mm_HandSolder, F.Cu at (182.9, 85.8)
- added R4: 330Ω 5% 1/8W, Resistor_SMD:R_0805_2012Metric_Pad1.20x1.40mm_HandSolder, F.Cu at (196.5, 67.0)
- added R5: 330Ω 5% 1/8W, Resistor_SMD:R_0805_2012Metric_Pad1.20x1.40mm_HandSolder, F.Cu at (175.1, 95.2)
- C1: value C -> 0.1u
- D1: value D_Filled -> PMLL4148L
- D2: value D_Zener -> 3.6V 1/2mW
- D5: renamed from D3; value LED -> Led Red
- J1: renamed from J2; value USB_A -> Pcb USB Type A
- J2: renamed from J1; value Conn_01x10_Socket -> Header
- R1: value R -> 1.5KΩ 5% 1/8W
- U1: footprint Package_SO:SOIC-8W_5.3x5.3mm_P1.27mm -> Package_SO:SOIC-8_5.3x5.3mm_P1.27mm
- moved D1 75.4 mm to (205.0, 88.7), turned to -90 degrees
- moved J1 74.2 mm to (201.8, 97.1), turned to 90 degrees
- moved J2 71.7 mm to (195.4, 60.5), turned to -90 degrees
- moved D2 69.2 mm to (198.5, 88.8), turned to -90 degrees
- moved R1 66.8 mm to (203.9, 84.1), turned to 180 degrees
- moved U1 53.4 mm to (184.2, 73.0)
- moved C1 37.7 mm to (166.2, 92.8), turned to 180 degrees
- moved D5 36.2 mm to (170.8, 98.6), turned to 180 degrees
Connections:
- C1 pad 1: unconnected-(C1-Pad1) -> +5V
- C1 pad 2: unconnected-(C1-Pad2) -> GND
- D1 pad 2: unconnected-(D1-A-Pad2) -> Net-(D1-A)
- D2 pad 1: unconnected-(D2-K-Pad1) -> Net-(D2-K)
- D2 pad 2: unconnected-(D2-A-Pad2) -> GND
- D5 pad 1: unconnected-(D3-K-Pad1) -> Net-(D5-K)
- D5 pad 2: unconnected-(D3-A-Pad2) -> +5V
- J1 pad 1: unconnected-(J2-VBUS-Pad1) -> Net-(D1-A)
- J1 pad 2: unconnected-(J2-D--Pad2) -> Net-(D2-K)
- J1 pad 3: unconnected-(J2-D+-Pad3) -> Net-(D3-K)
- J1 pad 4: unconnected-(J2-GND-Pad4) -> GND
- J2 pad 1: unconnected-(J1-Pin_1-Pad1) -> +5V
- J2 pad 2: unconnected-(J1-Pin_2-Pad2) -> GND
- J2 pad 4: unconnected-(J1-Pin_4-Pad4) -> Net-(J2-Pin_4)
- J2 pad 5: unconnected-(J1-Pin_5-Pad5) -> Net-(D4-A)
- J2 pad 6: unconnected-(J1-Pin_6-Pad6) -> Net-(J2-Pin_6)
- J2 pad 7: unconnected-(J1-Pin_7-Pad7) -> Net-(J2-Pin_7)
- J2 pad 8: unconnected-(J1-Pin_8-Pad8) -> Net-(J2-Pin_8)
- J2 pad 9: unconnected-(J1-Pin_9-Pad9) -> Net-(J2-Pin_9)
- R1 pad 2: unconnected-(R1-Pad2) -> Net-(D2-K)
- U1 pad 1: unconnected-(U1-~{RESET}/PB5-Pad1) -> Net-(J2-Pin_9)
- U1 pad 2: unconnected-(U1-XTAL1/PB3-Pad2) -> Net-(J2-Pin_7)
- U1 pad 3: unconnected-(U1-XTAL2/PB4-Pad3) -> Net-(J2-Pin_8)
- U1 pad 4: unconnected-(U1-GND-Pad4) -> GND
- U1 pad 5: unconnected-(U1-AREF/PB0-Pad5) -> Net-(J2-Pin_4)
- U1 pad 6: unconnected-(U1-PB1-Pad6) -> Net-(D4-A)
- U1 pad 7: unconnected-(U1-PB2-Pad7) -> Net-(J2-Pin_6)
- U1 pad 8: unconnected-(U1-VCC-Pad8) -> +5V
Routing:
- net GND: track 0.00 -> 128.1 mm
- net +5V: track 0.00 -> 117.7 mm
- net Net-(J2-Pin_8): track 0.00 -> 38.6 mm
- net Net-(D4-A): track 0.00 -> 38.4 mm
- net Net-(J2-Pin_7): track 0.00 -> 35.6 mm
- net Net-(J2-Pin_6): track 0.00 -> 26.3 mm
- net Net-(D3-K): track 0.00 -> 26.1 mm
- net Net-(D2-K): track 0.00 -> 19.1 mm
- net Net-(J2-Pin_4): track 0.00 -> 16.9 mm
- net Net-(J2-Pin_9): track 0.00 -> 12.9 mm
- net Net-(D1-A): track 0.00 -> 6.99 mm
- net Net-(D4-K): track 0.00 -> 5.62 mm
- net Net-(D5-K): track 0.00 -> 4.00 mm
Other:
- board outline added: 45 x 46.5 mm
